File: untitled.brd (EAGLE design)
At the start: 100 x 80 mm, 2 parts

Commit message: Add files via upload
Parts:
- removed D2: SFH482, led:SFH482
- added R1: (no value), resistor:0204V
- moved D1 11.7 mm to (22.9, 27.9)
Connections:
- new net N$1: D1.A, R1.1
- net GND: no longer D2.K
- net VCC: now also R1.2; no longer D1.A, D2.A
Routing:
- net GND: track 41.9 -> 0.00 mm
- net VCC: track 41.9 -> 0.00 mm
Changed lines of the file:
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@@
 <layer number="97" name="Info" color="7" fill="1" visible="no" active="no"/>
 <layer number="98" name="Guide" color="6" fill="1" visible="no" active="no"/>
+<layer number="99" name="SpiceOrder" color="5" fill="1" visible="no" active="no"/>
 </layers>
 <board>
@@
 </autorouter>
 <elements>
-<element name="D1" library="led" library_urn="urn:adsk.eagle:library:259" package="SFH482" package3d_urn="urn:adsk.eagle:package:15795/1" value="SFH482" x="25.4" y="39.37"/>
-<element name="D2" library="led" library_urn="urn:adsk.eagle:library:259" package="SFH482" package3d_urn="urn:adsk.eagle:package:15795/1" value="SFH482" x="60.96" y="54.61"/>
+<element name="D1" library="led" library_urn="urn:adsk.eagle:library:259" package="SFH482" package3d_urn="urn:adsk.eagle:package:15795/1" value="SFH482" x="22.86" y="27.94"/>
+<element name="R1" library="resistor" library_urn="urn:adsk.eagle:library:348" package="0204V" package3d_urn="urn:adsk.eagle:package:25948/1" value="" x="19.05" y="43.18" rot="R180"/>
 </elements>
 <signals>
 <signal name="VCC">
+<contactref element="R1" pad="2"/>
+</signal>
+<signal name="N$1">
+<contactref element="R1" pad="1"/>
 <contactref element="D1" pad="A"/>
-<contactref element="D2" pad="A"/>
-<wire x1="24.8412" y1="39.4716" x2="24.2316" y2="39.4716" width="0.1524" layer="1"/>
-<wire x1="39.9288" y1="54.5592" x2="24.8412" y2="39.4716" width="0.1524" layer="1"/>
-<wire x1="59.5884" y1="54.5592" x2="39.9288" y2="54.5592" width="0.1524" layer="1"/>
-<wire x1="24.2316" y1="39.4716" x2="24.13" y2="39.37" width="0.1524" layer="1"/>
-<wire x1="59.5884" y1="54.5592" x2="59.69" y2="54.61" width="0.1524" layer="1"/>
+<wire x1="20.32" y1="43.18" x2="21.59" y2="27.94" width="0" layer="19" extent="1-1"/>
 </signal>
 <signal name="GND">
 <contactref element="D1" pad="K"/>
-<contactref element="D2" pad="K"/>
-<wire x1="47.0916" y1="39.4716" x2="26.67" y2="39.4716" width="0.1524" layer="1"/>
-<wire x1="62.23" y1="54.61" x2="47.0916" y2="39.4716" width="0.1524" layer="1"/>
-<wire x1="26.67" y1="39.4716" x2="26.67" y2="39.37" width="0.1524" layer="1"/>
 </signal>
 </signals>
