File: micro_motor.brd (EAGLE design)
At the start: 100 x 80 mm, 56 parts

Commit message: Add files via upload
Parts:
- removed H1, H10, H11, H12, H13, H14, H15, H16, H17, H18, H19, H2, H20, H21, H22, H23, H24, H25, H26, H27, H28, H29, H3, H30, H31, H32, H33, H34, H35, H36, H37, H38, H39, H4, H40, H41, H42, H43, H44, H45, H46, H47, H48, H49, H5, H50, H51, H52, H53, H54, H55, H56, H6, H7, H8, H9: MOUNT-PAD-ROUND2.8, holes:2,8-PAD
- added 0, 1, 11, 12, 13, 14, 15, 16, 17, 18, 19, 2, 20, 21, 22, 23, 24, 25, 26, 27, 3, 4, 5, 6, 7, 8, 9, GND, GND_LEFT_ENC, GND_LEFT_MOTOR_DRIVER, GND_LEFT_MOTOR_DRIVER_2, GND_RIGHT_ENC, GND_RIGHT_MOTOR_DRIVER, GND_RIGHT_MOTOR_DRIVER_2, M!_LEFT_ENC, M1_ENABLE, M1_FORWARD_PWN, M1_LEFT, M1_LEFT_2, M1_REVERSE_PWN, M1_RIGHT_ENC, M2_ENABLE, M2_FORWARD_PWN, M2_LEFT_ENC, M2_REVERSE_PWN, M2_RIGHT, M2_RIGHT_2, M2_RIGHT_ENC, MOTOR_POWER_L, MOTOR_POWER_R, OUTA_LEFT_ENC, OUTA_RIGHT_ENC, OUTB_LEFT_ENC, OUTB_RIGHT_ENC, VCC_LEF_ENC, VCC_RIGHT_ENC: MOUNT-PAD-ROUND2.8, holes:2,8-PAD
Connections:
- net GND: now also GND_LEFT_ENC.B2,8, GND_LEFT_MOTOR_DRIVER.B2,8, GND_LEFT_MOTOR_DRIVER_2.B2,8, GND_RIGHT_ENC.B2,8, GND_RIGHT_MOTOR_DRIVER.B2,8, GND_RIGHT_MOTOR_DRIVER_2.B2,8; no longer H32.B2,8, H33.B2,8, H40.B2,8, H41.B2,8, H45.B2,8, H51.B2,8
- net N$1: now also 0.B2,8, OUTB_LEFT_ENC.B2,8; no longer H2.B2,8, H46.B2,8
- net N$10: now also M1_RIGHT_ENC.B2,8, M2_RIGHT_2.B2,8; no longer H42.B2,8, H56.B2,8
- net N$11: now also M!_LEFT_ENC.B2,8, M1_LEFT_2.B2,8; no longer H34.B2,8, H50.B2,8
- net N$12: now also 5.B2,8, M2_REVERSE_PWN.B2,8; no longer H38.B2,8, H7.B2,8
- net N$13: now also 23.B2,8, M2_ENABLE.B2,8; no longer H19.B2,8, H44.B2,8
- net N$14: now also 6.B2,8, M2_FORWARD_PWN.B2,8; no longer H43.B2,8, H8.B2,8
- net N$2: now also 1.B2,8, OUTA_LEFT_ENC.B2,8; no longer H3.B2,8, H47.B2,8
- net N$3: now also M1_LEFT.B2,8, M2_LEFT_ENC.B2,8; no longer H31.B2,8, H49.B2,8
- net N$4: now also 3.B2,8, M1_FORWARD_PWN.B2,8; no longer H30.B2,8, H5.B2,8
- net N$5: now also 4.B2,8, M1_REVERSE_PWN.B2,8; no longer H35.B2,8, H6.B2,8
- net N$6: now also 2.B2,8, M1_ENABLE.B2,8; no longer H29.B2,8, H4.B2,8
- net N$7: now also 8.B2,8, OUTA_RIGHT_ENC.B2,8; no longer H10.B2,8, H53.B2,8
- net N$8: now also M2_RIGHT.B2,8, M2_RIGHT_ENC.B2,8; no longer H39.B2,8, H55.B2,8
- net N$9: now also 7.B2,8, OUTB_RIGHT_ENC.B2,8; no longer H52.B2,8, H9.B2,8
- net VCC: now also 27.B2,8, MOTOR_POWER_L.B2,8, MOTOR_POWER_R.B2,8, VCC_LEF_ENC.B2,8, VCC_RIGHT_ENC.B2,8; no longer H15.B2,8, H36.B2,8, H37.B2,8, H48.B2,8, H54.B2,8

Commit message: Add files via upload
Parts:
- removed 27: MOUNT-PAD-ROUND2.8, holes:2,8-PAD
- added 10: MOUNT-PAD-ROUND2.8, holes:2,8-PAD
- moved GND 85.4 mm to (21.6, 67.3)
- moved 0 74.6 mm to (21.6, 59.7)
- moved 1 63.8 mm to (21.6, 52.1)
- moved 6 62.2 mm to (21.6, 16.5)
- moved 7 55.1 mm to (21.6, 8.89)
- moved 2 53.9 mm to (21.6, 45.7)
- moved 8 49.0 mm to (21.6, 2.54)
- moved 20 46.4 mm to (38.1, 24.1)
- moved 3 43.1 mm to (21.6, 38.1)
- moved 9 33.5 mm to (30.5, 2.54)
- moved 4 32.4 mm to (21.6, 30.5)
- moved 5 21.6 mm to (21.6, 22.9)
- moved 13 15.2 mm to (38.1, 31.8)
- moved 11 7.62 mm to (45.7, 16.5)
- moved 15 7.62 mm to (53.3, 31.8)
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Connections:
- net GND: now also GND.B2,8
- net N$13: now also 22.B2,8; no longer 23.B2,8
- net VCC: now also 26.B2,8; no longer 27.B2,8
