File: micro_ir_led.brd (EAGLE design)
At the start: 100 x 80 mm, 22 parts

Commit message: Add files via upload
Parts:
- removed R1, R2, R3: 330, rcl:0204V
- added RES_1, RES_2, RES_3: 330, rcl:0204V
- moved EMI_ANODE1 61.9 mm to (3.81, 66.0)
- moved REC_CATHODE2 57.3 mm to (91.4, 39.4)
- moved EMI_ANODE3 55.3 mm to (90.2, 66.0)
- moved REC_CATHODE 49.4 mm to (3.81, 36.8)
- moved R6 49.1 mm to (80.0, 41.9)
- moved A2 47.3 mm to (76.2, 5.08)
- moved EMI_CATHODE3 41.0 mm to (90.2, 55.9)
- moved REC_ANODE 39.5 mm to (3.81, 47.0)
- moved EMI_ANODE2 38.2 mm to (53.3, 74.9)
- moved R4 37.5 mm to (11.4, 41.9)
- moved EMI_CATHODE1 37.0 mm to (3.81, 55.9)
- moved A1 36.9 mm to (76.2, 12.7)
- moved REC_ANODE1 33.0 mm to (26.7, 76.2)
- moved REC_ANODE2 32.2 mm to (90.2, 47.0)
- moved EMI_CATHODE2 32.1 mm to (68.6, 74.9)
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Connections:
- removed net N$2: REC_ANODE2.B2,8
- net GND: now also RES_1.1, RES_2.1, RES_3.1; no longer R1.1, R2.1, R3.1
- net N$1: now also REC_ANODE2.B2,8
- net VCC: now also RES_1.2, RES_2.2, RES_3.2; no longer R1.2, R2.2, R3.2

Commit message: Add files via upload
Parts:
- added A3, A4, EMI_ANODE4, EMI_ANODE5, EMI_CATHODE4, EMI_CATHODE5, REC_ANODE3, REC_ANODE4, REC_CATHODE3, REC_CATHODE4: MOUNT-PAD-ROUND2.8, holes:2,8-PAD
- added R1, R2: 10k, resistor:0204V
- added RES_4, RES_5: 330, rcl:0204V
- moved A2 34.1 mm to (45.7, 20.3)
- moved A1 33.5 mm to (45.7, 26.7)
- moved A0 33.0 mm to (45.7, 33.0)
- moved 3.3V 32.1 mm to (45.7, 39.4)
- moved EMI_ANODE1 20.3 mm to (3.81, 45.7)
- moved EMI_ANODE3 19.2 mm to (92.7, 47.0)
- moved EMI_CATHODE3 15.5 mm to (92.7, 40.6)
- moved EMI_CATHODE1 15.2 mm to (3.81, 40.6)
- moved REC_ANODE2 14.2 mm to (92.7, 33.0)
- moved REC_CATHODE2 12.8 mm to (92.7, 26.7)
- moved REC_ANODE 12.7 mm to (3.81, 34.3)
- moved REC_CATHODE 8.89 mm to (3.81, 27.9)
- moved EMI_CATHODE2 6.48 mm to (62.2, 76.2)
- moved REC_ANODE1 5.08 mm to (31.8, 76.2)
- moved REC_CATHODE1 5.08 mm to (39.4, 76.2)
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Connections:
- removed net N$1: 3.3V.B2,8, REC_ANODE.B2,8, REC_ANODE1.B2,8, REC_ANODE2.B2,8
- new net N$2: 3.3V.B2,8, REC_ANODE.B2,8, REC_ANODE1.B2,8, REC_ANODE2.B2,8, REC_ANODE3.B2,8, REC_ANODE4.B2,8
- new net N$6: A3.B2,8, R1.2, REC_CATHODE3.B2,8
- new net N$7: A4.B2,8, R2.2, REC_CATHODE4.B2,8
- net GND: now also EMI_ANODE4.B2,8, EMI_ANODE5.B2,8, EMI_CATHODE4.B2,8, EMI_CATHODE5.B2,8, R1.1, R2.1, RES_4.1, RES_5.1
- net VCC: now also RES_4.2, RES_5.2

Commit message: Add files via upload
Parts:
- added A5, EMI_ANODE6, EMI_CATHODE6, REC_ANODE5, REC_CATHODE5: MOUNT-PAD-ROUND2.8, holes:2,8-PAD
- added R3: 10k, resistor:0204V
- added RES_6: 330, rcl:0204V
- moved RES_2 18.2 mm to (41.9, 71.1)
- moved EMI_CATHODE2 16.6 mm to (45.7, 77.5)
- moved EMI_ANODE2 15.3 mm to (39.4, 77.5)
- moved 3.3V 7.73 mm to (47.0, 47.0)
- moved A4 7.73 mm to (47.0, 14.0)
- moved A1 6.48 mm to (47.0, 33.0)
- moved A2 6.48 mm to (47.0, 26.7)
- moved REC_CATHODE3 6.48 mm to (47.0, 20.3)
- moved A0 6.48 mm to (47.0, 39.4)
- moved REC_CATHODE1 6.48 mm to (33.0, 77.5)
- moved REC_ANODE1 5.24 mm to (26.7, 77.5)
- moved R5 1.80 mm to (29.2, 71.1)
Connections:
- new net N$1: REC_ANODE5.B2,8
- new net N$8: A5.B2,8, R3.2, REC_CATHODE5.B2,8
- net GND: now also EMI_ANODE6.B2,8, EMI_CATHODE6.B2,8, R3.1, RES_6.1
- net VCC: now also RES_6.2
