File: micro_ir_led.sch (EAGLE design)
At the start: 22 parts

Commit message: Add files via upload
Parts:
- renumbered R1 to RES_1, R2 to RES_3, R3 to RES_2
Connections:
- removed net N$2: REC_ANODE2.MOUNT
- net N$1: now also REC_ANODE2.MOUNT
Changed lines of the file:
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@@
 <part name="GND3" library="supply1" library_urn="urn:adsk.eagle:library:371" deviceset="GND" device=""/>
 <part name="SUPPLY3" library="supply2" library_urn="urn:adsk.eagle:library:372" deviceset="VCC" device=""/>
-<part name="R3" library="rcl" library_urn="urn:adsk.eagle:library:334" deviceset="R-US_" device="0204/2V" package3d_urn="urn:adsk.eagle:package:23495/1" value="330"/>
+<part name="RES_2" library="rcl" library_urn="urn:adsk.eagle:library:334" deviceset="R-US_" device="0204/2V" package3d_urn="urn:adsk.eagle:package:23495/1" value="330"/>
 <part name="EMI_ANODE1" library="holes" library_urn="urn:adsk.eagle:library:237" deviceset="MOUNT-PAD-ROUND" device="2.8" package3d_urn="urn:adsk.eagle:package:14281/1"/>
 <part name="EMI_CATHODE1" library="holes" library_urn="urn:adsk.eagle:library:237" deviceset="MOUNT-PAD-ROUND" device="2.8" package3d_urn="urn:adsk.eagle:package:14281/1"/>
 <part name="GND1" library="supply1" library_urn="urn:adsk.eagle:library:371" deviceset="GND" device=""/>
 <part name="SUPPLY1" library="supply2" library_urn="urn:adsk.eagle:library:372" deviceset="VCC" device=""/>
-<part name="R1" library="rcl" library_urn="urn:adsk.eagle:library:334" deviceset="R-US_" device="0204/2V" package3d_urn="urn:adsk.eagle:package:23495/1" value="330"/>
+<part name="RES_1" library="rcl" library_urn="urn:adsk.eagle:library:334" deviceset="R-US_" device="0204/2V" package3d_urn="urn:adsk.eagle:package:23495/1" value="330"/>
 <part name="EMI_ANODE3" library="holes" library_urn="urn:adsk.eagle:library:237" deviceset="MOUNT-PAD-ROUND" device="2.8" package3d_urn="urn:adsk.eagle:package:14281/1"/>
 <part name="EMI_CATHODE3" library="holes" library_urn="urn:adsk.eagle:library:237" deviceset="MOUNT-PAD-ROUND" device="2.8" package3d_urn="urn:adsk.eagle:package:14281/1"/>
 <part name="GND2" library="supply1" library_urn="urn:adsk.eagle:library:371" deviceset="GND" device=""/>
 <part name="SUPPLY2" library="supply2" library_urn="urn:adsk.eagle:library:372" deviceset="VCC" device=""/>
-<part name="R2" library="rcl" library_urn="urn:adsk.eagle:library:334" deviceset="R-US_" device="0204/2V" package3d_urn="urn:adsk.eagle:package:23495/1" value="330"/>
+<part name="RES_3" library="rcl" library_urn="urn:adsk.eagle:library:334" deviceset="R-US_" device="0204/2V" package3d_urn="urn:adsk.eagle:package:23495/1" value="330"/>
 <part name="REC_ANODE" library="holes" library_urn="urn:adsk.eagle:library:237" deviceset="MOUNT-PAD-ROUND" device="2.8" package3d_urn="urn:adsk.eagle:package:14281/1"/>
 <part name="REC_CATHODE" library="holes" library_urn="urn:adsk.eagle:library:237" deviceset="MOUNT-PAD-ROUND" device="2.8" package3d_urn="urn:adsk.eagle:package:14281/1"/>
@@
 <instance part="GND3" gate="1" x="81.28" y="0"/>
 <instance part="SUPPLY3" gate="G$1" x="81.28" y="30.48"/>
-<instance part="R3" gate="G$1" x="-20.32" y="5.08"/>
+<instance part="RES_2" gate="G$1" x="-20.32" y="5.08"/>
 <instance part="EMI_ANODE1" gate="G$1" x="109.22" y="33.02"/>
 <instance part="EMI_CATHODE1" gate="G$1" x="154.94" y="33.02"/>
 <instance part="GND1" gate="1" x="223.52" y="-2.54"/>
 <instance part="SUPPLY1" gate="G$1" x="223.52" y="27.94"/>
-<instance part="R1" gate="G$1" x="121.92" y="2.54"/>
+<instance part="RES_1" gate="G$1" x="121.92" y="2.54"/>
 <instance part="EMI_ANODE3" gate="G$1" x="261.62" y="30.48"/>
 <instance part="EMI_CATHODE3" gate="G$1" x="307.34" y="30.48"/>
 <instance part="GND2" gate="1" x="375.92" y="-5.08"/>
 <instance part="SUPPLY2" gate="G$1" x="375.92" y="25.4"/>
-<instance part="R2" gate="G$1" x="274.32" y="0"/>
+<instance part="RES_3" gate="G$1" x="274.32" y="0"/>
 <instance part="REC_ANODE" gate="G$1" x="-27.94" y="-55.88"/>
 <instance part="REC_CATHODE" gate="G$1" x="7.62" y="-55.88"/>
@@
 <segment>
 <pinref part="SUPPLY3" gate="G$1" pin="VCC"/>
-<pinref part="R3" gate="G$1" pin="2"/>
+<pinref part="RES_2" gate="G$1" pin="2"/>
 <wire x1="81.28" y1="27.94" x2="-15.24" y2="27.94" width="0.1524" layer="91"/>
 <wire x1="-15.24" y1="27.94" x2="-15.24" y2="5.08" width="0.1524" layer="91"/>
@@
 <segment>
 <pinref part="SUPPLY1" gate="G$1" pin="VCC"/>
-<pinref part="R1" gate="G$1" pin="2"/>
+<pinref part="RES_1" gate="G$1" pin="2"/>
 <wire x1="223.52" y1="25.4" x2="127" y2="25.4" width="0.1524" layer="91"/>
 <wire x1="127" y1="25.4" x2="127" y2="2.54" width="0.1524" layer="91"/>
@@
 <segment>
 <pinref part="SUPPLY2" gate="G$1" pin="VCC"/>
-<pinref part="R2" gate="G$1" pin="2"/>
+<pinref part="RES_3" gate="G$1" pin="2"/>
 <wire x1="375.92" y1="22.86" x2="279.4" y2="22.86" width="0.1524" layer="91"/>
 <wire x1="279.4" y1="22.86" x2="279.4" y2="0" width="0.1524" layer="91"/>
@@
 <net name="GND" class="0">
 <segment>
-<pinref part="R3" gate="G$1" pin="1"/>
+<pinref part="RES_2" gate="G$1" pin="1"/>
 <pinref part="EMI_ANODE2" gate="G$1" pin="MOUNT"/>
 <wire x1="-25.4" y1="5.08" x2="-35.56" y2="5.08" width="0.1524" layer="91"/>
@@
 </segment>
 <segment>
-<pinref part="R1" gate="G$1" pin="1"/>
+<pinref part="RES_1" gate="G$1" pin="1"/>
 <pinref part="EMI_ANODE1" gate="G$1" pin="MOUNT"/>
 <wire x1="116.84" y1="2.54" x2="106.68" y2="2.54" width="0.1524" layer="91"/>
@@
 </segment>
 <segment>
-<pinref part="R2" gate="G$1" pin="1"/>
+<pinref part="RES_3" gate="G$1" pin="1"/>
 <pinref part="EMI_ANODE3" gate="G$1" pin="MOUNT"/>
 <wire x1="269.24" y1="0" x2="259.08" y2="0" width="0.1524" layer="91"/>
@@
 <wire x1="55.88" y1="-137.16" x2="55.88" y2="-55.88" width="0.1524" layer="91"/>
 <junction x="68.58" y="-137.16"/>
-</segment>
-</net>
-<net name="N$2" class="0">
-<segment>
 <pinref part="REC_ANODE2" gate="G$1" pin="MOUNT"/>
-<wire x1="73.66" y1="-137.16" x2="139.7" y2="-137.16" width="0.1524" layer="91"/>
+<wire x1="68.58" y1="-137.16" x2="139.7" y2="-137.16" width="0.1524" layer="91"/>
 <wire x1="139.7" y1="-137.16" x2="139.7" y2="-55.88" width="0.1524" layer="91"/>
 </segment>

Commit message: Add files via upload
Parts:
- added A3, A4, EMI_ANODE4, EMI_ANODE5, EMI_CATHODE4, EMI_CATHODE5, REC_ANODE3, REC_ANODE4, REC_CATHODE3, REC_CATHODE4: MOUNT-PAD-ROUND2.8, holes:MOUNT-PAD-ROUND2.8
- added R1, R2: 10k, resistor:R-US_0204/2V
- added RES_4, RES_5: 330, rcl:R-US_0204/2V
Connections:
- removed net N$1: 3.3V.MOUNT, REC_ANODE.MOUNT, REC_ANODE1.MOUNT, REC_ANODE2.MOUNT
- new net N$2: 3.3V.MOUNT, REC_ANODE.MOUNT, REC_ANODE1.MOUNT, REC_ANODE2.MOUNT, REC_ANODE3.MOUNT, REC_ANODE4.MOUNT
- new net N$6: A3.MOUNT, R1.2, REC_CATHODE3.MOUNT
- new net N$7: A4.MOUNT, R2.2, REC_CATHODE4.MOUNT
- net GND: now also EMI_ANODE4.MOUNT, EMI_ANODE5.MOUNT, EMI_CATHODE4.MOUNT, EMI_CATHODE5.MOUNT, R1.1, R2.1, RES_4.1, RES_5.1
- net VCC: now also RES_4.2, RES_5.2

Commit message: Add files via upload
Parts:
- added A5, EMI_ANODE6, EMI_CATHODE6, REC_ANODE5, REC_CATHODE5: MOUNT-PAD-ROUND2.8, holes:MOUNT-PAD-ROUND2.8
- added R3: 10k, resistor:R-US_0204/2V
- added RES_6: 330, rcl:R-US_0204/2V
Connections:
- new net N$1: REC_ANODE5.MOUNT
- new net N$8: A5.MOUNT, R3.2, REC_CATHODE5.MOUNT
- net GND: now also EMI_ANODE6.MOUNT, EMI_CATHODE6.MOUNT, R3.1, RES_6.1
- net VCC: now also RES_6.2
Changed lines of the file:
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@@
 <part name="A4" library="holes" library_urn="urn:adsk.eagle:library:237" deviceset="MOUNT-PAD-ROUND" device="2.8" package3d_urn="urn:adsk.eagle:package:14281/1"/>
 <part name="GND10" library="supply1" library_urn="urn:adsk.eagle:library:371" deviceset="GND" device=""/>
+<part name="EMI_ANODE6" library="holes" library_urn="urn:adsk.eagle:library:237" deviceset="MOUNT-PAD-ROUND" device="2.8" package3d_urn="urn:adsk.eagle:package:14281/1"/>
+<part name="EMI_CATHODE6" library="holes" library_urn="urn:adsk.eagle:library:237" deviceset="MOUNT-PAD-ROUND" device="2.8" package3d_urn="urn:adsk.eagle:package:14281/1"/>
+<part name="GND11" library="supply1" library_urn="urn:adsk.eagle:library:371" deviceset="GND" device=""/>
+<part name="SUPPLY6" library="supply2" library_urn="urn:adsk.eagle:library:372" deviceset="VCC" device=""/>
+<part name="RES_6" library="rcl" library_urn="urn:adsk.eagle:library:334" deviceset="R-US_" device="0204/2V" package3d_urn="urn:adsk.eagle:package:23495/1" value="330"/>
+<part name="REC_ANODE5" library="holes" library_urn="urn:adsk.eagle:library:237" deviceset="MOUNT-PAD-ROUND" device="2.8" package3d_urn="urn:adsk.eagle:package:14281/1"/>
+<part name="REC_CATHODE5" library="holes" library_urn="urn:adsk.eagle:library:237" deviceset="MOUNT-PAD-ROUND" device="2.8" package3d_urn="urn:adsk.eagle:package:14281/1"/>
+<part name="R3" library="resistor" library_urn="urn:adsk.eagle:library:348" deviceset="R-US_" device="0204/2V" package3d_urn="urn:adsk.eagle:package:25948/1" value="10k"/>
+<part name="A5" library="holes" library_urn="urn:adsk.eagle:library:237" deviceset="MOUNT-PAD-ROUND" device="2.8" package3d_urn="urn:adsk.eagle:package:14281/1"/>
+<part name="GND12" library="supply1" library_urn="urn:adsk.eagle:library:371" deviceset="GND" device=""/>
 </parts>
 <sheets>
@@
 <instance part="A4" gate="G$1" x="414.02" y="-78.74"/>
 <instance part="GND10" gate="1" x="414.02" y="-132.08"/>
+<instance part="EMI_ANODE6" gate="G$1" x="701.04" y="30.48"/>
+<instance part="EMI_CATHODE6" gate="G$1" x="746.76" y="30.48"/>
+<instance part="GND11" gate="1" x="815.34" y="-5.08"/>
+<instance part="SUPPLY6" gate="G$1" x="815.34" y="25.4"/>
+<instance part="RES_6" gate="G$1" x="713.74" y="0"/>
+<instance part="REC_ANODE5" gate="G$1" x="538.48" y="-58.42"/>
+<instance part="REC_CATHODE5" gate="G$1" x="574.04" y="-58.42"/>
+<instance part="R3" gate="G$1" x="553.72" y="-88.9"/>
+<instance part="A5" gate="G$1" x="571.5" y="-78.74"/>
+<instance part="GND12" gate="1" x="571.5" y="-132.08"/>
 </instances>
 <busses>
@@
 <wire x1="660.4" y1="22.86" x2="563.88" y2="22.86" width="0.1524" layer="91"/>
 <wire x1="563.88" y1="22.86" x2="563.88" y2="0" width="0.1524" layer="91"/>
+</segment>
+<segment>
+<pinref part="SUPPLY6" gate="G$1" pin="VCC"/>
+<pinref part="RES_6" gate="G$1" pin="2"/>
+<wire x1="815.34" y1="22.86" x2="718.82" y2="22.86" width="0.1524" layer="91"/>
+<wire x1="718.82" y1="22.86" x2="718.82" y2="0" width="0.1524" layer="91"/>
 </segment>
 </net>
@@
 <wire x1="391.16" y1="-88.9" x2="391.16" y2="-129.54" width="0.1524" layer="91"/>
 <wire x1="391.16" y1="-129.54" x2="414.02" y2="-129.54" width="0.1524" layer="91"/>
+</segment>
+<segment>
+<pinref part="RES_6" gate="G$1" pin="1"/>
+<pinref part="EMI_ANODE6" gate="G$1" pin="MOUNT"/>
+<wire x1="708.66" y1="0" x2="698.5" y2="0" width="0.1524" layer="91"/>
+<wire x1="698.5" y1="0" x2="698.5" y2="30.48" width="0.1524" layer="91"/>
+<pinref part="EMI_CATHODE6" gate="G$1" pin="MOUNT"/>
+<wire x1="698.5" y1="30.48" x2="744.22" y2="30.48" width="0.1524" layer="91"/>
+<junction x="698.5" y="30.48"/>
+<pinref part="GND11" gate="1" pin="GND"/>
+<wire x1="744.22" y1="30.48" x2="782.32" y2="30.48" width="0.1524" layer="91"/>
+<wire x1="782.32" y1="30.48" x2="815.34" y2="-2.54" width="0.1524" layer="91"/>
+<junction x="744.22" y="30.48"/>
+</segment>
+<segment>
+<pinref part="R3" gate="G$1" pin="1"/>
+<pinref part="GND12" gate="1" pin="GND"/>
+<wire x1="548.64" y1="-88.9" x2="548.64" y2="-129.54" width="0.1524" layer="91"/>
+<wire x1="548.64" y1="-129.54" x2="571.5" y2="-129.54" width="0.1524" layer="91"/>
 </segment>
 </net>
@@
 <junction x="68.58" y="-137.16"/>
 <pinref part="REC_ANODE2" gate="G$1" pin="MOUNT"/>
-<wire x1="68.58" y1="-137.16" x2="139.7" y2="-137.16" width="0.1524" layer="91"/>
 <wire x1="139.7" y1="-137.16" x2="139.7" y2="-55.88" width="0.1524" layer="91"/>
 <pinref part="REC_ANODE3" gate="G$1" pin="MOUNT"/>
 <wire x1="220.98" y1="-137.16" x2="220.98" y2="-55.88" width="0.1524" layer="91"/>
-<wire x1="68.58" y1="-137.16" x2="220.98" y2="-137.16" width="0.1524" layer="91"/>
+<wire x1="68.58" y1="-137.16" x2="139.7" y2="-137.16" width="0.1524" layer="91"/>
+<wire x1="139.7" y1="-137.16" x2="220.98" y2="-137.16" width="0.1524" layer="91"/>
 <wire x1="220.98" y1="-139.7" x2="220.98" y2="-137.16" width="0.1524" layer="91"/>
 <junction x="220.98" y="-137.16"/>
+<wire x1="139.7" y1="-137.16" x2="139.7" y2="-160.02" width="0.1524" layer="91"/>
+<junction x="139.7" y="-137.16"/>
+<wire x1="139.7" y1="-160.02" x2="68.58" y2="-160.02" width="0.1524" layer="91"/>
+<wire x1="66.04" y1="-160.02" x2="68.58" y2="-160.02" width="0.1524" layer="91"/>
+<wire x1="68.58" y1="-160.02" x2="68.58" y2="-149.86" width="0.1524" layer="91"/>
+<wire x1="220.98" y1="-137.16" x2="220.98" y2="-170.18" width="0.1524" layer="91"/>
+<wire x1="220.98" y1="-172.72" x2="220.98" y2="-170.18" width="0.1524" layer="91"/>
+<wire x1="220.98" y1="-170.18" x2="68.58" y2="-170.18" width="0.1524" layer="91"/>
+<wire x1="68.58" y1="-170.18" x2="68.58" y2="-160.02" width="0.1524" layer="91"/>
+<wire x1="68.58" y1="-149.86" x2="68.58" y2="-137.16" width="0.1524" layer="91"/>
+<wire x1="378.46" y1="-139.7" x2="378.46" y2="-149.86" width="0.1524" layer="91"/>
+<wire x1="378.46" y1="-149.86" x2="68.58" y2="-149.86" width="0.1524" layer="91"/>
+<junction x="378.46" y="-139.7"/>
+<junction x="68.58" y="-149.86"/>
 </segment>
 </net>
@@
 </segment>
 </net>
+<net name="N$1" class="0">
+<segment>
+<pinref part="REC_ANODE5" gate="G$1" pin="MOUNT"/>
+<wire x1="535.94" y1="-58.42" x2="535.94" y2="-139.7" width="0.1524" layer="91"/>
+<wire x1="535.94" y1="-139.7" x2="68.58" y2="-139.7" width="0.1524" layer="91"/>
+<wire x1="68.58" y1="-139.7" x2="68.58" y2="-142.24" width="0.1524" layer="91"/>
+<wire x1="68.58" y1="-139.7" x2="68.58" y2="-137.16" width="0.1524" layer="91"/>
+</segment>
+</net>
+<net name="N$8" class="0">
+<segment>
+<pinref part="REC_CATHODE5" gate="G$1" pin="MOUNT"/>
+<pinref part="A5" gate="G$1" pin="MOUNT"/>
+<wire x1="571.5" y1="-58.42" x2="571.5" y2="-78.74" width="0.1524" layer="91"/>
+<wire x1="571.5" y1="-78.74" x2="568.96" y2="-78.74" width="0.1524" layer="91"/>
+<pinref part="R3" gate="G$1" pin="2"/>
+<wire x1="568.96" y1="-78.74" x2="568.96" y2="-88.9" width="0.1524" layer="91"/>
+<wire x1="568.96" y1="-88.9" x2="558.8" y2="-88.9" width="0.1524" layer="91"/>
+<junction x="568.96" y="-78.74"/>
+</segment>
+</net>
