File: micromouse.sch (EAGLE design)
At the start: 24 parts

Commit message: Add files via upload
Parts:
- added C1: (no value), capacitor-wima:C2,5-3
Connections:
- removed net N$31: U$1.26, U$13.VCC, U$14.VCC, U$2.L_5V, U$2.R_5V
- new net GND: C1.2, R1.1, R2.2, R3.1, R4.1, R5.2, U$1.GND, U$10.EMI_CATHODE, U$11.EMI_CATHODE, U$12.EMI_CATHODE, U$13.GND, U$14.GND, U$2.L_GND_1, U$2.L_GND_2, U$2.R_GND_1, U$2.R_GND_2, U$8.EMI_CATHODE, U$9.EMI_CATHODE
- net N$30: now also C1.1, U$1.26, U$13.VCC, U$14.VCC, U$2.L_5V, U$2.R_5V; no longer R1.1, R2.2, R3.1, R4.1, R5.2, U$1.GND, U$10.EMI_CATHODE, U$11.EMI_CATHODE, U$12.EMI_CATHODE, U$13.GND, U$14.GND, U$2.L_GND_1, U$2.L_GND_2, U$2.R_GND_1, U$2.R_GND_2, U$8.EMI_CATHODE, U$9.EMI_CATHODE
Changed lines of the file:
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@@
 <part name="U$13" library="MOTOR_ENCODER" deviceset="MOTOR_ENCODER" device=""/>
 <part name="U$14" library="MOTOR_ENCODER" deviceset="MOTOR_ENCODER" device=""/>
+<part name="GND1" library="supply1" library_urn="urn:adsk.eagle:library:371" deviceset="GND" device=""/>
+<part name="C1" library="capacitor-wima" library_urn="urn:adsk.eagle:library:116" deviceset="C" device="2,5-3" package3d_urn="urn:adsk.eagle:package:5436/1"/>
 </parts>
 <sheets>
@@
 <instance part="U$13" gate="G$1" x="-111.76" y="27.94"/>
 <instance part="U$14" gate="G$1" x="213.36" y="12.7"/>
+<instance part="GND1" gate="1" x="20.32" y="-22.86"/>
+<instance part="C1" gate="G$1" x="76.2" y="71.12"/>
 </instances>
 <busses>
@@
 </segment>
 </net>
-<net name="N$30" class="0">
+<net name="N$26" class="0">
+<segment>
+<pinref part="U$14" gate="G$1" pin="OUTB"/>
+<wire x1="210.82" y1="22.86" x2="215.9" y2="22.86" width="0.1524" layer="91"/>
+<wire x1="215.9" y1="22.86" x2="215.9" y2="48.26" width="0.1524" layer="91"/>
+<wire x1="215.9" y1="48.26" x2="167.64" y2="48.26" width="0.1524" layer="91"/>
+<wire x1="167.64" y1="48.26" x2="167.64" y2="30.48" width="0.1524" layer="91"/>
+<pinref part="U$1" gate="G$1" pin="20"/>
+<wire x1="167.64" y1="30.48" x2="104.14" y2="30.48" width="0.1524" layer="91"/>
+</segment>
+</net>
+<net name="N$28" class="0">
+<segment>
+<pinref part="U$14" gate="G$1" pin="OUTA"/>
+<wire x1="210.82" y1="20.32" x2="218.44" y2="20.32" width="0.1524" layer="91"/>
+<wire x1="218.44" y1="20.32" x2="218.44" y2="53.34" width="0.1524" layer="91"/>
+<wire x1="218.44" y1="53.34" x2="170.18" y2="53.34" width="0.1524" layer="91"/>
+<wire x1="170.18" y1="53.34" x2="170.18" y2="33.02" width="0.1524" layer="91"/>
+<pinref part="U$1" gate="G$1" pin="21"/>
+<wire x1="170.18" y1="33.02" x2="104.14" y2="33.02" width="0.1524" layer="91"/>
+</segment>
+</net>
+<net name="N$6" class="0">
+<segment>
+<pinref part="U$14" gate="G$1" pin="M2"/>
+<wire x1="210.82" y1="15.24" x2="223.52" y2="15.24" width="0.1524" layer="91"/>
+<wire x1="223.52" y1="15.24" x2="223.52" y2="-7.62" width="0.1524" layer="91"/>
+<wire x1="223.52" y1="-7.62" x2="60.96" y2="-7.62" width="0.1524" layer="91"/>
+<wire x1="60.96" y1="-7.62" x2="60.96" y2="20.32" width="0.1524" layer="91"/>
+<pinref part="U$2" gate="G$1" pin="R_M2_2"/>
+<wire x1="60.96" y1="20.32" x2="25.4" y2="20.32" width="0.1524" layer="91"/>
+</segment>
+</net>
+<net name="N$32" class="0">
+<segment>
+<pinref part="U$14" gate="G$1" pin="M1"/>
+<wire x1="210.82" y1="12.7" x2="210.82" y2="7.62" width="0.1524" layer="91"/>
+<wire x1="210.82" y1="7.62" x2="88.9" y2="7.62" width="0.1524" layer="91"/>
+<wire x1="88.9" y1="7.62" x2="88.9" y2="5.08" width="0.1524" layer="91"/>
+<wire x1="88.9" y1="5.08" x2="45.72" y2="5.08" width="0.1524" layer="91"/>
+<pinref part="U$2" gate="G$1" pin="R_M2_1"/>
+<wire x1="45.72" y1="5.08" x2="45.72" y2="27.94" width="0.1524" layer="91"/>
+<wire x1="45.72" y1="27.94" x2="25.4" y2="27.94" width="0.1524" layer="91"/>
+</segment>
+</net>
+<net name="GND" class="0">
 <segment>
 <pinref part="U$14" gate="G$1" pin="GND"/>
@@
 <wire x1="58.42" y1="-5.08" x2="53.34" y2="-5.08" width="0.1524" layer="91"/>
 <junction x="53.34" y="-5.08"/>
-</segment>
-</net>
-<net name="N$26" class="0">
-<segment>
-<pinref part="U$14" gate="G$1" pin="OUTB"/>
-<wire x1="210.82" y1="22.86" x2="215.9" y2="22.86" width="0.1524" layer="91"/>
-<wire x1="215.9" y1="22.86" x2="215.9" y2="48.26" width="0.1524" layer="91"/>
-<wire x1="215.9" y1="48.26" x2="167.64" y2="48.26" width="0.1524" layer="91"/>
-<wire x1="167.64" y1="48.26" x2="167.64" y2="30.48" width="0.1524" layer="91"/>
-<pinref part="U$1" gate="G$1" pin="20"/>
-<wire x1="167.64" y1="30.48" x2="104.14" y2="30.48" width="0.1524" layer="91"/>
-</segment>
-</net>
-<net name="N$28" class="0">
-<segment>
-<pinref part="U$14" gate="G$1" pin="OUTA"/>
-<wire x1="210.82" y1="20.32" x2="218.44" y2="20.32" width="0.1524" layer="91"/>
-<wire x1="218.44" y1="20.32" x2="218.44" y2="53.34" width="0.1524" layer="91"/>
-<wire x1="218.44" y1="53.34" x2="170.18" y2="53.34" width="0.1524" layer="91"/>
-<wire x1="170.18" y1="53.34" x2="170.18" y2="33.02" width="0.1524" layer="91"/>
-<pinref part="U$1" gate="G$1" pin="21"/>
-<wire x1="170.18" y1="33.02" x2="104.14" y2="33.02" width="0.1524" layer="91"/>
-</segment>
-</net>
-<net name="N$31" class="0">
-<segment>
+<pinref part="GND1" gate="1" pin="GND"/>
+<pinref part="C1" gate="G$1" pin="2"/>
+<wire x1="76.2" y1="66.04" x2="78.74" y2="66.04" width="0.1524" layer="91"/>
+<wire x1="78.74" y1="66.04" x2="78.74" y2="45.72" width="0.1524" layer="91"/>
+<junction x="78.74" y="45.72"/>
+</segment>
+</net>
+<net name="N$30" class="0">
+<segment>
+<pinref part="C1" gate="G$1" pin="1"/>
+<wire x1="76.2" y1="73.66" x2="81.28" y2="73.66" width="0.1524" layer="91"/>
+<wire x1="81.28" y1="73.66" x2="81.28" y2="53.34" width="0.1524" layer="91"/>
+<wire x1="81.28" y1="53.34" x2="106.68" y2="53.34" width="0.1524" layer="91"/>
 <pinref part="U$14" gate="G$1" pin="VCC"/>
 <wire x1="210.82" y1="17.78" x2="228.6" y2="17.78" width="0.1524" layer="91"/>
@@
 <wire x1="228.6" y1="-40.64" x2="124.46" y2="-40.64" width="0.1524" layer="91"/>
 <pinref part="U$1" gate="G$1" pin="26"/>
-<wire x1="104.14" y1="45.72" x2="121.92" y2="45.72" width="0.1524" layer="91"/>
+<wire x1="104.14" y1="45.72" x2="106.68" y2="45.72" width="0.1524" layer="91"/>
+<wire x1="106.68" y1="45.72" x2="121.92" y2="45.72" width="0.1524" layer="91"/>
 <wire x1="121.92" y1="45.72" x2="121.92" y2="-20.32" width="0.1524" layer="91"/>
 <wire x1="121.92" y1="-20.32" x2="124.46" y2="-20.32" width="0.1524" layer="91"/>
@@
 <wire x1="124.46" y1="-40.64" x2="124.46" y2="-20.32" width="0.1524" layer="91"/>
 <junction x="124.46" y="-20.32"/>
-</segment>
-</net>
-<net name="N$6" class="0">
-<segment>
-<pinref part="U$14" gate="G$1" pin="M2"/>
-<wire x1="210.82" y1="15.24" x2="223.52" y2="15.24" width="0.1524" layer="91"/>
-<wire x1="223.52" y1="15.24" x2="223.52" y2="-7.62" width="0.1524" layer="91"/>
-<wire x1="223.52" y1="-7.62" x2="60.96" y2="-7.62" width="0.1524" layer="91"/>
-<wire x1="60.96" y1="-7.62" x2="60.96" y2="20.32" width="0.1524" layer="91"/>
-<pinref part="U$2" gate="G$1" pin="R_M2_2"/>
-<wire x1="60.96" y1="20.32" x2="25.4" y2="20.32" width="0.1524" layer="91"/>
-</segment>
-</net>
-<net name="N$32" class="0">
-<segment>
-<pinref part="U$14" gate="G$1" pin="M1"/>
-<wire x1="210.82" y1="12.7" x2="210.82" y2="7.62" width="0.1524" layer="91"/>
-<wire x1="210.82" y1="7.62" x2="88.9" y2="7.62" width="0.1524" layer="91"/>
-<wire x1="88.9" y1="7.62" x2="88.9" y2="5.08" width="0.1524" layer="91"/>
-<wire x1="88.9" y1="5.08" x2="45.72" y2="5.08" width="0.1524" layer="91"/>
-<pinref part="U$2" gate="G$1" pin="R_M2_1"/>
-<wire x1="45.72" y1="5.08" x2="45.72" y2="27.94" width="0.1524" layer="91"/>
-<wire x1="45.72" y1="27.94" x2="25.4" y2="27.94" width="0.1524" layer="91"/>
-</segment>
-</net>
+<wire x1="106.68" y1="53.34" x2="106.68" y2="45.72" width="0.1524" layer="91"/>
+<junction x="106.68" y="45.72"/>
+</segment>
+</net>

Commit message: Add files via upload
Changed lines of the file:
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@@
 <wire x1="99.06" y1="142.24" x2="60.96" y2="142.24" width="0.1524" layer="91"/>
 <wire x1="60.96" y1="142.24" x2="17.78" y2="142.24" width="0.1524" layer="91"/>
-<wire x1="17.78" y1="142.24" x2="-25.4" y2="142.24" width="0.1524" layer="91"/>
-<wire x1="-25.4" y1="142.24" x2="-104.14" y2="142.24" width="0.1524" layer="91"/>
+<wire x1="17.78" y1="142.24" x2="-27.94" y2="142.24" width="0.1524" layer="91"/>
+<wire x1="-27.94" y1="142.24" x2="-104.14" y2="142.24" width="0.1524" layer="91"/>
 <wire x1="-104.14" y1="142.24" x2="-104.14" y2="104.14" width="0.1524" layer="91"/>
 <wire x1="-104.14" y1="104.14" x2="-40.64" y2="104.14" width="0.1524" layer="91"/>
 <pinref part="U$3" gate="G$1" pin="REC_ANODE"/>
 <wire x1="-40.64" y1="104.14" x2="-40.64" y2="109.22" width="0.1524" layer="91"/>
-<wire x1="-25.4" y1="142.24" x2="-25.4" y2="101.6" width="0.1524" layer="91"/>
-<junction x="-25.4" y="142.24"/>
+<wire x1="-27.94" y1="142.24" x2="-27.94" y2="101.6" width="0.1524" layer="91"/>
+<junction x="-27.94" y="142.24"/>
 <pinref part="U$4" gate="G$1" pin="REC_ANODE"/>
-<wire x1="-25.4" y1="101.6" x2="2.54" y2="101.6" width="0.1524" layer="91"/>
+<wire x1="-27.94" y1="101.6" x2="2.54" y2="101.6" width="0.1524" layer="91"/>
 <wire x1="2.54" y1="101.6" x2="2.54" y2="109.22" width="0.1524" layer="91"/>
 <wire x1="17.78" y1="142.24" x2="17.78" y2="104.14" width="0.1524" layer="91"/>

Commit message: Add files via upload
Changed lines of the file:
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@@
-</segment>
-</net>
-<net name="N$23" class="0">
-<segment>
-<pinref part="U$1" gate="G$1" pin="24"/>
-<wire x1="104.14" y1="40.64" x2="223.52" y2="40.64" width="0.1524" layer="91"/>
-<wire x1="223.52" y1="40.64" x2="223.52" y2="119.38" width="0.1524" layer="91"/>
-<wire x1="223.52" y1="119.38" x2="185.42" y2="119.38" width="0.1524" layer="91"/>
-<wire x1="185.42" y1="119.38" x2="182.88" y2="119.38" width="0.1524" layer="91"/>
-<wire x1="185.42" y1="119.38" x2="185.42" y2="142.24" width="0.1524" layer="91"/>
-<junction x="185.42" y="119.38"/>
-<wire x1="185.42" y1="142.24" x2="99.06" y2="142.24" width="0.1524" layer="91"/>
-<wire x1="99.06" y1="142.24" x2="60.96" y2="142.24" width="0.1524" layer="91"/>
-<wire x1="60.96" y1="142.24" x2="17.78" y2="142.24" width="0.1524" layer="91"/>
-<wire x1="17.78" y1="142.24" x2="-27.94" y2="142.24" width="0.1524" layer="91"/>
-<wire x1="-27.94" y1="142.24" x2="-104.14" y2="142.24" width="0.1524" layer="91"/>
-<wire x1="-104.14" y1="142.24" x2="-104.14" y2="104.14" width="0.1524" layer="91"/>
-<wire x1="-104.14" y1="104.14" x2="-40.64" y2="104.14" width="0.1524" layer="91"/>
-<pinref part="U$3" gate="G$1" pin="REC_ANODE"/>
-<wire x1="-40.64" y1="104.14" x2="-40.64" y2="109.22" width="0.1524" layer="91"/>
-<wire x1="-27.94" y1="142.24" x2="-27.94" y2="101.6" width="0.1524" layer="91"/>
-<junction x="-27.94" y="142.24"/>
-<pinref part="U$4" gate="G$1" pin="REC_ANODE"/>
-<wire x1="-27.94" y1="101.6" x2="2.54" y2="101.6" width="0.1524" layer="91"/>
-<wire x1="2.54" y1="101.6" x2="2.54" y2="109.22" width="0.1524" layer="91"/>
-<wire x1="17.78" y1="142.24" x2="17.78" y2="104.14" width="0.1524" layer="91"/>
-<wire x1="17.78" y1="104.14" x2="40.64" y2="104.14" width="0.1524" layer="91"/>
-<junction x="17.78" y="142.24"/>
-<pinref part="U$5" gate="G$1" pin="REC_ANODE"/>
-<wire x1="40.64" y1="104.14" x2="40.64" y2="109.22" width="0.1524" layer="91"/>
-<wire x1="60.96" y1="142.24" x2="60.96" y2="104.14" width="0.1524" layer="91"/>
-<wire x1="60.96" y1="104.14" x2="81.28" y2="104.14" width="0.1524" layer="91"/>
-<pinref part="U$6" gate="G$1" pin="REC_ANODE"/>
-<wire x1="81.28" y1="104.14" x2="81.28" y2="109.22" width="0.1524" layer="91"/>
-<wire x1="99.06" y1="142.24" x2="99.06" y2="104.14" width="0.1524" layer="91"/>
-<junction x="99.06" y="142.24"/>
-<wire x1="99.06" y1="104.14" x2="124.46" y2="104.14" width="0.1524" layer="91"/>
-<pinref part="U$7" gate="G$1" pin="REC_ANODE"/>
-<wire x1="124.46" y1="104.14" x2="124.46" y2="109.22" width="0.1524" layer="91"/>
-<junction x="60.96" y="142.24"/>
 </segment>
 </net>
@@
 </segment>
 </net>
+<net name="N$36" class="0">
+<segment>
+<pinref part="U$7" gate="G$1" pin="REC_ANODE"/>
+<wire x1="124.46" y1="104.14" x2="124.46" y2="109.22" width="0.1524" layer="91"/>
+<wire x1="99.06" y1="160.02" x2="99.06" y2="104.14" width="0.1524" layer="91"/>
+<wire x1="99.06" y1="104.14" x2="124.46" y2="104.14" width="0.1524" layer="91"/>
+<pinref part="U$6" gate="G$1" pin="REC_ANODE"/>
+<wire x1="81.28" y1="104.14" x2="81.28" y2="109.22" width="0.1524" layer="91"/>
+<wire x1="60.96" y1="154.94" x2="60.96" y2="104.14" width="0.1524" layer="91"/>
+<wire x1="60.96" y1="104.14" x2="81.28" y2="104.14" width="0.1524" layer="91"/>
+<pinref part="U$5" gate="G$1" pin="REC_ANODE"/>
+<wire x1="40.64" y1="104.14" x2="40.64" y2="109.22" width="0.1524" layer="91"/>
+<wire x1="17.78" y1="149.86" x2="17.78" y2="104.14" width="0.1524" layer="91"/>
+<wire x1="17.78" y1="104.14" x2="40.64" y2="104.14" width="0.1524" layer="91"/>
+<pinref part="U$4" gate="G$1" pin="REC_ANODE"/>
+<wire x1="2.54" y1="101.6" x2="2.54" y2="109.22" width="0.1524" layer="91"/>
+<wire x1="-27.94" y1="101.6" x2="2.54" y2="101.6" width="0.1524" layer="91"/>
+<wire x1="-27.94" y1="101.6" x2="-27.94" y2="147.32" width="0.1524" layer="91"/>
+<pinref part="U$3" gate="G$1" pin="REC_ANODE"/>
+<wire x1="-40.64" y1="104.14" x2="-40.64" y2="109.22" width="0.1524" layer="91"/>
+<wire x1="-104.14" y1="152.4" x2="-104.14" y2="104.14" width="0.1524" layer="91"/>
+<wire x1="-104.14" y1="104.14" x2="-40.64" y2="104.14" width="0.1524" layer="91"/>
+<pinref part="U$1" gate="G$1" pin="24"/>
+<wire x1="104.14" y1="40.64" x2="223.52" y2="40.64" width="0.1524" layer="91"/>
+<wire x1="223.52" y1="40.64" x2="223.52" y2="119.38" width="0.1524" layer="91"/>
+<wire x1="223.52" y1="119.38" x2="200.66" y2="119.38" width="0.1524" layer="91"/>
+<wire x1="200.66" y1="119.38" x2="195.58" y2="119.38" width="0.1524" layer="91"/>
+<wire x1="195.58" y1="119.38" x2="193.04" y2="119.38" width="0.1524" layer="91"/>
+<wire x1="193.04" y1="119.38" x2="190.5" y2="119.38" width="0.1524" layer="91"/>
+<wire x1="190.5" y1="119.38" x2="185.42" y2="119.38" width="0.1524" layer="91"/>
+<wire x1="185.42" y1="119.38" x2="182.88" y2="119.38" width="0.1524" layer="91"/>
+<wire x1="-104.14" y1="152.4" x2="185.42" y2="152.4" width="0.1524" layer="91"/>
+<wire x1="185.42" y1="152.4" x2="185.42" y2="119.38" width="0.1524" layer="91"/>
+<junction x="185.42" y="119.38"/>
+<wire x1="-27.94" y1="147.32" x2="190.5" y2="147.32" width="0.1524" layer="91"/>
+<wire x1="190.5" y1="147.32" x2="190.5" y2="119.38" width="0.1524" layer="91"/>
+<junction x="190.5" y="119.38"/>
+<wire x1="17.78" y1="149.86" x2="193.04" y2="149.86" width="0.1524" layer="91"/>
+<wire x1="193.04" y1="149.86" x2="193.04" y2="119.38" width="0.1524" layer="91"/>
+<junction x="193.04" y="119.38"/>
+<wire x1="60.96" y1="154.94" x2="195.58" y2="154.94" width="0.1524" layer="91"/>
+<wire x1="195.58" y1="154.94" x2="195.58" y2="119.38" width="0.1524" layer="91"/>
+<junction x="195.58" y="119.38"/>
+<wire x1="99.06" y1="160.02" x2="200.66" y2="160.02" width="0.1524" layer="91"/>
+<wire x1="200.66" y1="160.02" x2="200.66" y2="119.38" width="0.1524" layer="91"/>
+<junction x="200.66" y="119.38"/>
+</segment>
+</net>

Commit message: Add files via upload
Parts:
- added U$15: VOLTAGE_REGULATOR, VOLTAGE_REGULATOR:VOLTAGE_REGULATOR
Connections:
- net GND: now also U$15.GND
- net N$30: now also U$15.VOUT
Changed lines of the file:
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@@
 <part name="GND1" library="supply1" library_urn="urn:adsk.eagle:library:371" deviceset="GND" device=""/>
 <part name="C1" library="capacitor-wima" library_urn="urn:adsk.eagle:library:116" deviceset="C" device="2,5-3" package3d_urn="urn:adsk.eagle:package:5436/1"/>
+<part name="U$15" library="VOLTAGE_REGULATOR" deviceset="VOLTAGE_REGULATOR" device=""/>
 </parts>
 <sheets>
@@
 <instance part="GND1" gate="1" x="20.32" y="-22.86"/>
 <instance part="C1" gate="G$1" x="76.2" y="71.12"/>
+<instance part="U$15" gate="G$1" x="129.54" y="-60.96"/>
 </instances>
 <busses>
@@
 <wire x1="17.78" y1="-7.62" x2="53.34" y2="-7.62" width="0.1524" layer="91"/>
 <junction x="53.34" y="-7.62"/>
-<wire x1="25.4" y1="-20.32" x2="20.32" y2="-20.32" width="0.1524" layer="91"/>
+<wire x1="25.4" y1="-20.32" x2="22.86" y2="-20.32" width="0.1524" layer="91"/>
+<wire x1="22.86" y1="-20.32" x2="20.32" y2="-20.32" width="0.1524" layer="91"/>
 <wire x1="58.42" y1="-5.08" x2="53.34" y2="-5.08" width="0.1524" layer="91"/>
 <junction x="53.34" y="-5.08"/>
@@
 <wire x1="78.74" y1="66.04" x2="78.74" y2="45.72" width="0.1524" layer="91"/>
 <junction x="78.74" y="45.72"/>
+<pinref part="U$15" gate="G$1" pin="GND"/>
+<wire x1="114.3" y1="-48.26" x2="114.3" y2="-45.72" width="0.1524" layer="91"/>
+<wire x1="114.3" y1="-45.72" x2="22.86" y2="-45.72" width="0.1524" layer="91"/>
+<wire x1="22.86" y1="-45.72" x2="22.86" y2="-20.32" width="0.1524" layer="91"/>
+<junction x="22.86" y="-20.32"/>
 </segment>
 </net>
@@
 <wire x1="106.68" y1="53.34" x2="106.68" y2="45.72" width="0.1524" layer="91"/>
 <junction x="106.68" y="45.72"/>
-</segment>
-</net>
+<pinref part="U$15" gate="G$1" pin="VOUT"/>
+<wire x1="111.76" y1="-48.26" x2="111.76" y2="-22.86" width="0.1524" layer="91"/>
+<wire x1="111.76" y1="-22.86" x2="149.86" y2="-22.86" width="0.1524" layer="91"/>
+<wire x1="149.86" y1="-22.86" x2="149.86" y2="-20.32" width="0.1524" layer="91"/>
+</segment>
+</net>
