File: micromouse.brd (EAGLE design)
At the start: 100 x 80 mm, 22 parts

Commit message: Add files via upload
Parts:
- added U$13, U$14: MOTOR_ENCODER, MOTOR_ENCODER:MOTOR_ENCODER
Connections:
- new net N$25: U$13.P$2, U$2.L_M1_1
- new net N$26: U$1.20, U$14.P$5
- new net N$27: U$1.13, U$13.P$4
- new net N$29: U$1.19, U$13.P$5
- new net N$3: U$13.P$3, U$2.L_M1_2
- new net N$30: R1.1, R2.2, R3.1, R4.1, R5.2, U$1.GND, U$10.2, U$11.2, U$12.2, U$13.P$1, U$14.P$1, U$2.L_GND_1, U$2.L_GND_2, U$2.R_GND_1, U$2.R_GND_2, U$8.2, U$9.2
- new net N$31: U$1.26, U$13.P$6, U$14.P$6, U$2.L_5V, U$2.R_5V
- new net N$32: U$14.P$2, U$2.R_M2_1
- net N$28: now also U$1.21, U$14.P$4; no longer R1.1, R2.2, R3.1, R4.1, R5.2, U$1.GND, U$10.2, U$11.2, U$12.2, U$2.L_GND_1, U$2.L_GND_2, U$2.R_GND_1, U$2.R_GND_2, U$8.2, U$9.2
- net N$6: now also U$14.P$3, U$2.R_M2_2; no longer U$1.26, U$2.L_5V, U$2.R_5V
Changed lines of the file:
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@@
 <attribute name="SPICEPREFIX" value="R" x="31.75" y="50.8" size="1.778" layer="27" display="off"/>
 </element>
+<element name="U$13" library="MOTOR_ENCODER" package="MOTOR_ENCODER" value="MOTOR_ENCODER" x="-5.08" y="10.16"/>
+<element name="U$14" library="MOTOR_ENCODER" package="MOTOR_ENCODER" value="MOTOR_ENCODER" x="-16.51" y="10.16"/>
 </elements>
 <signals>
@@
 <contactref element="U$1" pad="2"/>
 <wire x1="41.91" y1="16.51" x2="41.91" y2="38.1" width="0" layer="19" extent="1-1"/>
-</signal>
-<signal name="N$6">
-<contactref element="U$1" pad="26"/>
-<contactref element="U$2" pad="L_5V"/>
-<contactref element="U$2" pad="R_5V"/>
-<wire x1="49.53" y1="16.51" x2="49.53" y2="41.91" width="0" layer="19" extent="1-1"/>
-<wire x1="41.91" y1="7.62" x2="49.53" y2="16.51" width="0" layer="19" extent="1-1"/>
 </signal>
 <signal name="N$8">
@@
 <wire x1="49.53" y1="31.75" x2="29.21" y2="50.8" width="0" layer="19" extent="1-1"/>
 </signal>
-<signal name="N$28">
+<signal name="N$3">
+<contactref element="U$13" pad="P$3"/>
+<contactref element="U$2" pad="L_M1_2"/>
+<wire x1="-6.35" y1="10.16" x2="41.91" y2="10.16" width="0" layer="19" extent="1-1"/>
+</signal>
+<signal name="N$25">
+<contactref element="U$13" pad="P$2"/>
+<contactref element="U$2" pad="L_M1_1"/>
+<wire x1="-6.35" y1="11.43" x2="41.91" y2="13.97" width="0" layer="19" extent="1-1"/>
+</signal>
+<signal name="N$27">
+<contactref element="U$13" pad="P$4"/>
+<contactref element="U$1" pad="13"/>
+<wire x1="-6.35" y1="8.89" x2="49.53" y2="25.4" width="0" layer="19" extent="1-1"/>
+</signal>
+<signal name="N$29">
+<contactref element="U$13" pad="P$5"/>
+<contactref element="U$1" pad="19"/>
+<wire x1="-6.35" y1="7.62" x2="49.53" y2="33.02" width="0" layer="19" extent="1-1"/>
+</signal>
+<signal name="N$30">
+<contactref element="U$14" pad="P$1"/>
 <contactref element="R1" pad="1"/>
 <contactref element="U$1" pad="GND"/>
@@
 <contactref element="R5" pad="2"/>
 <contactref element="R2" pad="2"/>
+<contactref element="U$13" pad="P$1"/>
 <wire x1="93.98" y1="49.53" x2="93.98" y2="57.15" width="0" layer="19" extent="1-1"/>
 <wire x1="77.47" y1="71.12" x2="93.98" y2="57.15" width="0" layer="19" extent="1-1"/>
@@
 <wire x1="49.53" y1="12.7" x2="41.91" y2="12.7" width="0" layer="19" extent="1-1"/>
 <wire x1="49.53" y1="11.43" x2="49.53" y2="12.7" width="0" layer="19" extent="1-1"/>
+<wire x1="-6.35" y1="12.7" x2="21.59" y2="50.8" width="0" layer="19" extent="1-1"/>
+<wire x1="-17.78" y1="12.7" x2="-6.35" y2="12.7" width="0" layer="19" extent="1-1"/>
+</signal>
+<signal name="N$26">
+<contactref element="U$14" pad="P$5"/>
+<contactref element="U$1" pad="20"/>
+<wire x1="-17.78" y1="7.62" x2="49.53" y2="34.29" width="0" layer="19" extent="1-1"/>
+</signal>
+<signal name="N$28">
+<contactref element="U$14" pad="P$4"/>
+<contactref element="U$1" pad="21"/>
+<wire x1="-17.78" y1="8.89" x2="49.53" y2="35.56" width="0" layer="19" extent="1-1"/>
+</signal>
+<signal name="N$31">
+<contactref element="U$14" pad="P$6"/>
+<contactref element="U$1" pad="26"/>
+<contactref element="U$2" pad="L_5V"/>
+<contactref element="U$2" pad="R_5V"/>
+<contactref element="U$13" pad="P$6"/>
+<wire x1="49.53" y1="16.51" x2="49.53" y2="41.91" width="0" layer="19" extent="1-1"/>
+<wire x1="41.91" y1="7.62" x2="49.53" y2="16.51" width="0" layer="19" extent="1-1"/>
+<wire x1="-6.35" y1="6.35" x2="41.91" y2="7.62" width="0" layer="19" extent="1-1"/>
+<wire x1="-17.78" y1="6.35" x2="-6.35" y2="6.35" width="0" layer="19" extent="1-1"/>
+</signal>
+<signal name="N$6">
+<contactref element="U$14" pad="P$3"/>
+<contactref element="U$2" pad="R_M2_2"/>
+<wire x1="-17.78" y1="10.16" x2="49.53" y2="10.16" width="0" layer="19" extent="1-1"/>
+</signal>
+<signal name="N$32">
+<contactref element="U$14" pad="P$2"/>
+<contactref element="U$2" pad="R_M2_1"/>
+<wire x1="-17.78" y1="11.43" x2="49.53" y2="13.97" width="0" layer="19" extent="1-1"/>
 </signal>
 </signals>

Commit message: Add files via upload
Parts:
- moved U$14 95.8 mm to (78.7, 20.3)
- moved U$13 24.1 mm to (17.8, 17.8)
Changed lines of the file:
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@@
 <attribute name="SPICEPREFIX" value="R" x="31.75" y="50.8" size="1.778" layer="27" display="off"/>
 </element>
-<element name="U$13" library="MOTOR_ENCODER" package="MOTOR_ENCODER" value="MOTOR_ENCODER" x="-5.08" y="10.16"/>
-<element name="U$14" library="MOTOR_ENCODER" package="MOTOR_ENCODER" value="MOTOR_ENCODER" x="-16.51" y="10.16"/>
+<element name="U$13" library="MOTOR_ENCODER" package="MOTOR_ENCODER" value="MOTOR_ENCODER" x="17.78" y="17.78"/>
+<element name="U$14" library="MOTOR_ENCODER" package="MOTOR_ENCODER" value="MOTOR_ENCODER" x="78.74" y="20.32"/>
 </elements>
 <signals>
@@
 <contactref element="U$13" pad="P$3"/>
 <contactref element="U$2" pad="L_M1_2"/>
-<wire x1="-6.35" y1="10.16" x2="41.91" y2="10.16" width="0" layer="19" extent="1-1"/>
+<wire x1="16.51" y1="17.78" x2="41.91" y2="10.16" width="0" layer="19" extent="1-1"/>
 </signal>
 <signal name="N$25">
 <contactref element="U$13" pad="P$2"/>
 <contactref element="U$2" pad="L_M1_1"/>
-<wire x1="-6.35" y1="11.43" x2="41.91" y2="13.97" width="0" layer="19" extent="1-1"/>
+<wire x1="16.51" y1="19.05" x2="41.91" y2="13.97" width="0" layer="19" extent="1-1"/>
 </signal>
 <signal name="N$27">
 <contactref element="U$13" pad="P$4"/>
 <contactref element="U$1" pad="13"/>
-<wire x1="-6.35" y1="8.89" x2="49.53" y2="25.4" width="0" layer="19" extent="1-1"/>
+<wire x1="16.51" y1="16.51" x2="49.53" y2="25.4" width="0" layer="19" extent="1-1"/>
 </signal>
 <signal name="N$29">
 <contactref element="U$13" pad="P$5"/>
 <contactref element="U$1" pad="19"/>
-<wire x1="-6.35" y1="7.62" x2="49.53" y2="33.02" width="0" layer="19" extent="1-1"/>
+<wire x1="16.51" y1="15.24" x2="49.53" y2="33.02" width="0" layer="19" extent="1-1"/>
 </signal>
 <signal name="N$30">
@@
 <wire x1="49.53" y1="12.7" x2="41.91" y2="12.7" width="0" layer="19" extent="1-1"/>
 <wire x1="49.53" y1="11.43" x2="49.53" y2="12.7" width="0" layer="19" extent="1-1"/>
-<wire x1="-6.35" y1="12.7" x2="21.59" y2="50.8" width="0" layer="19" extent="1-1"/>
-<wire x1="-17.78" y1="12.7" x2="-6.35" y2="12.7" width="0" layer="19" extent="1-1"/>
+<wire x1="16.51" y1="20.32" x2="21.59" y2="50.8" width="0" layer="19" extent="1-1"/>
+<wire x1="77.47" y1="22.86" x2="16.51" y2="20.32" width="0" layer="19" extent="1-1"/>
 </signal>
 <signal name="N$26">
 <contactref element="U$14" pad="P$5"/>
 <contactref element="U$1" pad="20"/>
-<wire x1="-17.78" y1="7.62" x2="49.53" y2="34.29" width="0" layer="19" extent="1-1"/>
+<wire x1="77.47" y1="17.78" x2="49.53" y2="34.29" width="0" layer="19" extent="1-1"/>
 </signal>
 <signal name="N$28">
 <contactref element="U$14" pad="P$4"/>
 <contactref element="U$1" pad="21"/>
-<wire x1="-17.78" y1="8.89" x2="49.53" y2="35.56" width="0" layer="19" extent="1-1"/>
+<wire x1="77.47" y1="19.05" x2="49.53" y2="35.56" width="0" layer="19" extent="1-1"/>
 </signal>
 <signal name="N$31">
@@
 <wire x1="49.53" y1="16.51" x2="49.53" y2="41.91" width="0" layer="19" extent="1-1"/>
 <wire x1="41.91" y1="7.62" x2="49.53" y2="16.51" width="0" layer="19" extent="1-1"/>
-<wire x1="-6.35" y1="6.35" x2="41.91" y2="7.62" width="0" layer="19" extent="1-1"/>
-<wire x1="-17.78" y1="6.35" x2="-6.35" y2="6.35" width="0" layer="19" extent="1-1"/>
+<wire x1="16.51" y1="13.97" x2="41.91" y2="7.62" width="0" layer="19" extent="1-1"/>
+<wire x1="77.47" y1="16.51" x2="16.51" y2="13.97" width="0" layer="19" extent="1-1"/>
 </signal>
 <signal name="N$6">
 <contactref element="U$14" pad="P$3"/>
 <contactref element="U$2" pad="R_M2_2"/>
-<wire x1="-17.78" y1="10.16" x2="49.53" y2="10.16" width="0" layer="19" extent="1-1"/>
+<wire x1="77.47" y1="20.32" x2="49.53" y2="10.16" width="0" layer="19" extent="1-1"/>
 </signal>
 <signal name="N$32">
 <contactref element="U$14" pad="P$2"/>
 <contactref element="U$2" pad="R_M2_1"/>
-<wire x1="-17.78" y1="11.43" x2="49.53" y2="13.97" width="0" layer="19" extent="1-1"/>
+<wire x1="77.47" y1="21.59" x2="49.53" y2="13.97" width="0" layer="19" extent="1-1"/>
 </signal>
 </signals>

Commit message: Add files via upload
Parts:
- moved U$4 91.5 mm to (97.8, 54.6)
- moved U$5 87.7 mm to (96.5, 68.6)
- moved U$11 87.7 mm to (6.35, 59.7)
- moved U$9 64.8 mm to (6.35, 72.4)
- moved R8 52.4 mm to (86.4, 72.4)
- moved R1 39.6 mm to (86.4, 54.6)
- moved R2 36.4 mm to (86.4, 68.6)
- moved R5 31.8 mm to (57.1, 69.8)
- moved R9 31.8 mm to (14.0, 59.7)
- moved R6 30.2 mm to (47.0, 71.1)
- moved R10 29.2 mm to (86.4, 59.7)
- moved R3 25.7 mm to (14.0, 54.6)
- moved U$10 19.1 mm to (96.5, 72.4)
- moved U$7 15.7 mm to (57.1, 76.2)
- moved R4 15.5 mm to (21.6, 66.0)
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
Commit message: Add files via upload
Parts:
- added C1: (no value), capacitor-wima:C2.5-3
Connections:
- removed net N$31: U$1.26, U$13.P$6, U$14.P$6, U$2.L_5V, U$2.R_5V
- new net GND: C1.2, R1.1, R2.2, R3.1, R4.1, R5.2, U$1.GND, U$10.2, U$11.2, U$12.2, U$13.P$1, U$14.P$1, U$2.L_GND_1, U$2.L_GND_2, U$2.R_GND_1, U$2.R_GND_2, U$8.2, U$9.2
- net N$30: now also C1.1, U$1.26, U$13.P$6, U$14.P$6, U$2.L_5V, U$2.R_5V; no longer R1.1, R2.2, R3.1, R4.1, R5.2, U$1.GND, U$10.2, U$11.2, U$12.2, U$13.P$1, U$14.P$1, U$2.L_GND_1, U$2.L_GND_2, U$2.R_GND_1, U$2.R_GND_2, U$8.2, U$9.2
Changed lines of the file:
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@@
 <element name="U$13" library="MOTOR_ENCODER" package="MOTOR_ENCODER" value="MOTOR_ENCODER" x="17.78" y="17.78"/>
 <element name="U$14" library="MOTOR_ENCODER" package="MOTOR_ENCODER" value="MOTOR_ENCODER" x="78.74" y="20.32"/>
+<element name="C1" library="capacitor-wima" library_urn="urn:adsk.eagle:library:116" package="C2.5-3" package3d_urn="urn:adsk.eagle:package:5436/1" value="" x="8.89" y="-8.89"/>
 </elements>
 <signals>
@@
 <contactref element="U$8" pad="1"/>
 <contactref element="R6" pad="2"/>
-<wire x1="49.53" y1="71.12" x2="45.72" y2="76.2" width="0" layer="19" extent="1-1"/>
+<wire x1="45.72" y1="76.2" x2="49.53" y2="71.12" width="0" layer="19" extent="1-1"/>
 </signal>
 <signal name="N$10">
 <contactref element="U$1" pad="0"/>
 <contactref element="R6" pad="1"/>
-<wire x1="41.91" y1="40.64" x2="44.45" y2="71.12" width="0" layer="19" extent="1-1"/>
+<wire x1="44.45" y1="71.12" x2="41.91" y2="40.64" width="0" layer="19" extent="1-1"/>
 </signal>
 <signal name="N$11">
@@
 <contactref element="U$1" pad="7"/>
 <contactref element="R7" pad="2"/>
-<wire x1="41.91" y1="31.75" x2="24.13" y2="71.12" width="0" layer="19" extent="1-1"/>
+<wire x1="24.13" y1="71.12" x2="41.91" y2="31.75" width="0" layer="19" extent="1-1"/>
 </signal>
 <signal name="N$13">
@@
 <contactref element="U$12" pad="1"/>
 <contactref element="R10" pad="1"/>
-<wire x1="83.82" y1="59.69" x2="96.52" y2="59.69" width="0" layer="19" extent="1-1"/>
+<wire x1="96.52" y1="59.69" x2="83.82" y2="59.69" width="0" layer="19" extent="1-1"/>
 </signal>
 <signal name="N$18">
@@
 <contactref element="U$1" pad="18"/>
 <contactref element="R5" pad="1"/>
-<wire x1="54.61" y1="69.85" x2="57.15" y2="76.2" width="0" layer="19" extent="1-1"/>
+<wire x1="57.15" y1="76.2" x2="54.61" y2="69.85" width="0" layer="19" extent="1-1"/>
 <wire x1="49.53" y1="31.75" x2="54.61" y2="69.85" width="0" layer="19" extent="1-1"/>
 </signal>
@@
 <wire x1="16.51" y1="15.24" x2="49.53" y2="33.02" width="0" layer="19" extent="1-1"/>
 </signal>
-<signal name="N$30">
+<signal name="N$26">
+<contactref element="U$14" pad="P$5"/>
+<contactref element="U$1" pad="20"/>
+<wire x1="49.53" y1="34.29" x2="77.47" y2="17.78" width="0" layer="19" extent="1-1"/>
+</signal>
+<signal name="N$28">
+<contactref element="U$14" pad="P$4"/>
+<contactref element="U$1" pad="21"/>
+<wire x1="49.53" y1="35.56" x2="77.47" y2="19.05" width="0" layer="19" extent="1-1"/>
+</signal>
+<signal name="N$6">
+<contactref element="U$14" pad="P$3"/>
+<contactref element="U$2" pad="R_M2_2"/>
+<wire x1="49.53" y1="10.16" x2="77.47" y2="20.32" width="0" layer="19" extent="1-1"/>
+</signal>
+<signal name="N$32">
+<contactref element="U$14" pad="P$2"/>
+<contactref element="U$2" pad="R_M2_1"/>
+<wire x1="49.53" y1="13.97" x2="77.47" y2="21.59" width="0" layer="19" extent="1-1"/>
+</signal>
+<signal name="GND">
 <contactref element="U$14" pad="P$1"/>
 <contactref element="R1" pad="1"/>
@@
 <contactref element="R2" pad="2"/>
 <contactref element="U$13" pad="P$1"/>
+<contactref element="C1" pad="2"/>
 <wire x1="88.9" y1="68.58" x2="96.52" y2="72.39" width="0" layer="19" extent="1-1"/>
 <wire x1="97.79" y1="59.69" x2="88.9" y2="68.58" width="0" layer="19" extent="1-1"/>
@@
 <wire x1="16.51" y1="20.32" x2="41.91" y2="12.7" width="0" layer="19" extent="1-1"/>
 <wire x1="41.91" y1="41.91" x2="41.91" y2="12.7" width="0" layer="19" extent="1-1"/>
-</signal>
-<signal name="N$26">
-<contactref element="U$14" pad="P$5"/>
-<contactref element="U$1" pad="20"/>
-<wire x1="49.53" y1="34.29" x2="77.47" y2="17.78" width="0" layer="19" extent="1-1"/>
-</signal>
-<signal name="N$28">
-<contactref element="U$14" pad="P$4"/>
-<contactref element="U$1" pad="21"/>
-<wire x1="49.53" y1="35.56" x2="77.47" y2="19.05" width="0" layer="19" extent="1-1"/>
-</signal>
-<signal name="N$31">
+<wire x1="10.16" y1="-8.89" x2="16.51" y2="20.32" width="0" layer="19" extent="1-1"/>
+</signal>
+<signal name="N$30">
+<contactref element="C1" pad="1"/>
 <contactref element="U$14" pad="P$6"/>
 <contactref element="U$1" pad="26"/>
@@
 <wire x1="49.53" y1="41.91" x2="49.53" y2="16.51" width="0" layer="19" extent="1-1"/>
 <wire x1="16.51" y1="13.97" x2="41.91" y2="7.62" width="0" layer="19" extent="1-1"/>
-</signal>
-<signal name="N$6">
-<contactref element="U$14" pad="P$3"/>
-<contactref element="U$2" pad="R_M2_2"/>
-<wire x1="49.53" y1="10.16" x2="77.47" y2="20.32" width="0" layer="19" extent="1-1"/>
-</signal>
-<signal name="N$32">
-<contactref element="U$14" pad="P$2"/>
-<contactref element="U$2" pad="R_M2_1"/>
-<wire x1="49.53" y1="13.97" x2="77.47" y2="21.59" width="0" layer="19" extent="1-1"/>
+<wire x1="7.62" y1="-8.89" x2="16.51" y2="13.97" width="0" layer="19" extent="1-1"/>
 </signal>
 </signals>

Commit message: Add files via upload
Parts:
- moved C1 48.2 mm to (24.1, 36.8)
Changed lines of the file:
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@@
 <element name="U$13" library="MOTOR_ENCODER" package="MOTOR_ENCODER" value="MOTOR_ENCODER" x="17.78" y="17.78"/>
 <element name="U$14" library="MOTOR_ENCODER" package="MOTOR_ENCODER" value="MOTOR_ENCODER" x="78.74" y="20.32"/>
-<element name="C1" library="capacitor-wima" library_urn="urn:adsk.eagle:library:116" package="C2.5-3" package3d_urn="urn:adsk.eagle:package:5436/1" value="" x="8.89" y="-8.89"/>
+<element name="C1" library="capacitor-wima" library_urn="urn:adsk.eagle:library:116" package="C2.5-3" package3d_urn="urn:adsk.eagle:package:5436/1" value="" x="24.13" y="36.83"/>
 </elements>
 <signals>
@@
 <wire x1="16.51" y1="20.32" x2="41.91" y2="12.7" width="0" layer="19" extent="1-1"/>
 <wire x1="41.91" y1="41.91" x2="41.91" y2="12.7" width="0" layer="19" extent="1-1"/>
-<wire x1="10.16" y1="-8.89" x2="16.51" y2="20.32" width="0" layer="19" extent="1-1"/>
+<wire x1="25.4" y1="36.83" x2="16.51" y2="20.32" width="0" layer="19" extent="1-1"/>
 </signal>
 <signal name="N$30">
@@
 <wire x1="49.53" y1="41.91" x2="49.53" y2="16.51" width="0" layer="19" extent="1-1"/>
 <wire x1="16.51" y1="13.97" x2="41.91" y2="7.62" width="0" layer="19" extent="1-1"/>
-<wire x1="7.62" y1="-8.89" x2="16.51" y2="13.97" width="0" layer="19" extent="1-1"/>
+<wire x1="22.86" y1="36.83" x2="16.51" y2="13.97" width="0" layer="19" extent="1-1"/>
 </signal>
 </signals>

Commit message: Add files via upload
Parts:
- moved C1 9.25 mm to (15.2, 34.3), turned to 90 degrees
- moved R4 9.25 mm to (12.7, 68.6)
- moved R7 9.25 mm to (12.7, 73.7)
- moved U$14 6.48 mm to (85.1, 19.1)
- moved R6 5.39 mm to (43.2, 67.3)
- moved U$4 5.39 mm to (94.0, 50.8)
- moved U$12 4.58 mm to (94.0, 57.1)
- moved R1 3.81 mm to (86.4, 50.8)
- moved U$8 3.81 mm to (43.2, 76.2)
- moved U$13 3.81 mm to (14.0, 17.8)
- moved U$1 3.59 mm to (48.3, 36.8)
- moved R5 2.84 mm to (58.4, 67.3)
- moved U$10 2.84 mm to (94.0, 73.7)
- moved U$5 2.84 mm to (94.0, 67.3)
- moved R10 2.54 mm to (86.4, 57.1)
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Routing:
- net GND: track 0.00 -> 428.1 mm, vias 0 -> 1
- net N$36: track 0.00 -> 156.3 mm, vias 0 -> 2
- net N$30: track 0.00 -> 142.6 mm
- net N$29: track 0.00 -> 84.7 mm
- net N$21: track 0.00 -> 77.5 mm, vias 0 -> 2
- net N$14: track 0.00 -> 72.5 mm, vias 0 -> 7
- net N$18: track 0.00 -> 67.7 mm, vias 0 -> 1
- net N$20: track 0.00 -> 59.6 mm, vias 0 -> 2
- net N$24: track 0.00 -> 58.6 mm, vias 0 -> 4
- net N$2: track 0.00 -> 52.3 mm, vias 0 -> 4
- net N$12: track 0.00 -> 51.6 mm
- net N$28: track 0.00 -> 49.8 mm, vias 0 -> 4
- net N$27: track 0.00 -> 49.0 mm, vias 0 -> 2
- net N$7: track 0.00 -> 48.7 mm, vias 0 -> 2
- net N$19: track 0.00 -> 48.6 mm
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
Commit message: Add files via upload
Parts:
- added U$15: VOLTAGE_REGULATOR, VOLTAGE_REGULATOR:VOLTAGE_REGULATOR
Connections:
- net GND: now also U$15.P$2
- net N$30: now also U$15.P$1
Routing:
- net GND: track 428.1 -> 446.5 mm
- net N$30: track 142.6 -> 153.2 mm
Changed lines of the file:
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@@
 <element name="U$14" library="MOTOR_ENCODER" package="MOTOR_ENCODER" value="MOTOR_ENCODER" x="85.09" y="19.05"/>
 <element name="C1" library="capacitor-wima" library_urn="urn:adsk.eagle:library:116" package="C2.5-3" package3d_urn="urn:adsk.eagle:package:5436/1" value="" x="15.24" y="34.29" rot="R90"/>
+<element name="U$15" library="VOLTAGE_REGULATOR" package="VOLTAGE_REGULATOR" value="VOLTAGE_REGULATOR" x="5.08" y="5.08"/>
 </elements>
 <signals>
@@
 <via x="33.02" y="12.7" extent="1-16" drill="0.35"/>
 <wire x1="33.02" y1="12.7" x2="15.24" y2="35.56" width="0.1524" layer="16"/>
+<contactref element="U$15" pad="P$2"/>
+<wire x1="12.0513125" y1="19.8326" x2="12.2126" y2="19.8326" width="0.1524" layer="16"/>
+<wire x1="12.2126" y1="19.8326" x2="12.7" y2="20.32" width="0.1524" layer="16"/>
+<wire x1="5.08" y1="5.08" x2="5.08" y2="12.8612875" width="0.1524" layer="16"/>
+<wire x1="5.08" y1="12.8612875" x2="12.0513125" y2="19.8326" width="0.1524" layer="16"/>
 </signal>
 <signal name="N$30">
@@
 <wire x1="56.9887125" y1="6.35" x2="59.69" y2="9.0512875" width="0.1524" layer="1"/>
 <wire x1="45.72" y1="6.35" x2="56.9887125" y2="6.35" width="0.1524" layer="1"/>
+<contactref element="U$15" pad="P$1"/>
+<wire x1="3.81" y1="5.08" x2="4.2974" y2="5.5674" width="0.1524" layer="1"/>
+<wire x1="4.2974" y1="5.5674" x2="4.2974" y2="5.7286875" width="0.1524" layer="1"/>
+<wire x1="4.2974" y1="5.7286875" x2="7.4587125" y2="8.89" width="0.1524" layer="1"/>
+<wire x1="7.4587125" y1="8.89" x2="12.7" y2="8.89" width="0.1524" layer="1"/>
 </signal>
 <signal name="N$36">

Commit message: Add files via upload
Routing:
- net N$36: track 156.3 -> 190.8 mm, vias 2 -> 8
- net N$24: track 58.6 -> 72.3 mm, vias 4 -> 7
- net N$13: track 0.00 -> 10.3 mm, vias 0 -> 1
- net N$11: track 0.00 -> 7.59 mm, vias 0 -> 2
- net N$15: track 13.5 -> 7.19 mm
- net N$4: track 38.9 -> 41.7 mm, vias 4 -> 5
- net N$21: track 77.5 -> 76.6 mm
- net N$29: track 84.7 -> 85.3 mm, vias 0 -> 1
