File: MICRO_2/micromouse.brd (EAGLE design)
At the start: 100 x 80 mm, 27 parts

Commit message: make 5v and 3.3v traces 12 mil and just dont worry about gound plane
Routing:
- net M2_L: track 60.9 -> 347.5 mm
- net N$9: track 239.8 -> 0.00 mm
- net N$6: track 196.0 -> 0.00 mm
- net N$5: track 193.5 -> 0.00 mm
- net M2_ENABLE: track 138.2 -> 0.00 mm
- net N$12: track 135.6 -> 14.8 mm
- net N$19: track 0.00 -> 112.5 mm
- net N$25: track 216.5 -> 112.2 mm, vias 1 -> 0
- net 3.3V_VCC: track 0.00 -> 86.9 mm
- net N$22: track 80.0 -> 0.00 mm
- net 5V_VCC: track 0.00 -> 72.8 mm, vias 0 -> 4
- net N$24: track 72.6 -> 0.00 mm
- net M1_L: track 72.0 -> 0.00 mm
- net N$8: track 194.7 -> 123.0 mm
- net N$21: track 62.6 -> 127.1 mm
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
Commit message: Add files via upload
Routing:
- net GND: track 46.1 -> 325.0 mm, vias 0 -> 12
- net 3.3V_VCC: track 86.9 -> 198.6 mm, vias 0 -> 4
- net 5V_VCC: track 72.8 -> 98.9 mm, vias 4 -> 5
