File: MICRO_4/micromouse.sch (EAGLE design)
At the start: 35 parts

Commit message: added motor_bracket lbr. need to fix dimension so motor bracket is in mm and board is in mil
Parts:
- added U$24, U$25: MOTOR_BRACKET, MOTOR_BRACKET:MOTOR_BRACKET
Changed lines of the file:
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@@
 <part name="R11" library="rcl" library_urn="urn:adsk.eagle:library:334" deviceset="R-US_" device="0207/10" package3d_urn="urn:adsk.eagle:package:23491/1" value="330"/>
 <part name="R12" library="rcl" library_urn="urn:adsk.eagle:library:334" deviceset="R-US_" device="0207/10" package3d_urn="urn:adsk.eagle:package:23491/1" value="10K"/>
+<part name="U$24" library="MOTOR_BRACKET" deviceset="MOTOR_BRACKET" device=""/>
+<part name="U$25" library="MOTOR_BRACKET" deviceset="MOTOR_BRACKET" device=""/>
 </parts>
 <sheets>
@@
 <instance part="R11" gate="G$1" x="-393.7" y="-20.32"/>
 <instance part="R12" gate="G$1" x="-360.68" y="-20.32"/>
+<instance part="U$24" gate="G$1" x="-381" y="-91.44"/>
+<instance part="U$25" gate="G$1" x="-381" y="-109.22"/>
 </instances>
 <busses>
@@
 <pinref part="U$10" gate="G$1" pin="GND"/>
 <wire x1="93.98" y1="-15.24" x2="58.42" y2="-15.24" width="0.1524" layer="91"/>
-<wire x1="58.42" y1="-15.24" x2="58.42" y2="-12.7" width="0.1524" layer="91"/>
-<wire x1="58.42" y1="-12.7" x2="58.42" y2="-10.16" width="0.1524" layer="91"/>
+<wire x1="58.42" y1="-15.24" x2="58.42" y2="-10.16" width="0.1524" layer="91"/>
 <wire x1="58.42" y1="-15.24" x2="58.42" y2="-40.64" width="0.1524" layer="91"/>
 <wire x1="58.42" y1="-40.64" x2="33.02" y2="-40.64" width="0.1524" layer="91"/>
@@
 <wire x1="83.82" y1="116.84" x2="83.82" y2="33.02" width="0.1524" layer="91"/>
 <junction x="83.82" y="33.02"/>
-<wire x1="76.2" y1="-12.7" x2="58.42" y2="-12.7" width="0.1524" layer="91"/>
-<junction x="58.42" y="-12.7"/>
 <wire x1="81.28" y1="124.46" x2="81.28" y2="33.02" width="0.1524" layer="91"/>
 <junction x="81.28" y="33.02"/>

Commit message: changed emitter library to make them more consistent
Parts:
- removed U$20, U$21: THRU_HOLE, THRU_HOLE:THRU_HOLE
- removed U$24, U$25: MOTOR_BRACKET, MOTOR_BRACKET:MOTOR_BRACKET
- U$18, U$19: value THRU_HOLE -> MOTOR_BRACKET; device THRU_HOLE:THRU_HOLE -> MOTOR_BRACKET:MOTOR_BRACKET
Changed lines of the file:
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@@
 <part name="R9" library="rcl" library_urn="urn:adsk.eagle:library:334" deviceset="R-US_" device="0207/10" package3d_urn="urn:adsk.eagle:package:23491/1" value="330"/>
 <part name="R10" library="rcl" library_urn="urn:adsk.eagle:library:334" deviceset="R-US_" device="0207/10" package3d_urn="urn:adsk.eagle:package:23491/1" value="10K"/>
-<part name="U$18" library="THRU_HOLE" deviceset="THRU_HOLE" device=""/>
-<part name="U$19" library="THRU_HOLE" deviceset="THRU_HOLE" device=""/>
-<part name="U$20" library="THRU_HOLE" deviceset="THRU_HOLE" device=""/>
-<part name="U$21" library="THRU_HOLE" deviceset="THRU_HOLE" device=""/>
 <part name="U$22" library="IR_EMITTER" deviceset="IR_EMITTER" device=""/>
 <part name="U$23" library="IR_RECIEVER" deviceset="IR_RECIEVER" device=""/>
 <part name="R11" library="rcl" library_urn="urn:adsk.eagle:library:334" deviceset="R-US_" device="0207/10" package3d_urn="urn:adsk.eagle:package:23491/1" value="330"/>
 <part name="R12" library="rcl" library_urn="urn:adsk.eagle:library:334" deviceset="R-US_" device="0207/10" package3d_urn="urn:adsk.eagle:package:23491/1" value="10K"/>
-<part name="U$24" library="MOTOR_BRACKET" deviceset="MOTOR_BRACKET" device=""/>
-<part name="U$25" library="MOTOR_BRACKET" deviceset="MOTOR_BRACKET" device=""/>
+<part name="U$18" library="MOTOR_BRACKET" deviceset="MOTOR_BRACKET" device=""/>
+<part name="U$19" library="MOTOR_BRACKET" deviceset="MOTOR_BRACKET" device=""/>
 </parts>
 <sheets>
@@
 <instance part="R9" gate="G$1" x="-309.88" y="-20.32"/>
 <instance part="R10" gate="G$1" x="-276.86" y="-20.32"/>
-<instance part="U$18" gate="G$1" x="-289.56" y="-111.76"/>
-<instance part="U$19" gate="G$1" x="-289.56" y="-124.46"/>
-<instance part="U$20" gate="G$1" x="-289.56" y="-139.7"/>
-<instance part="U$21" gate="G$1" x="-289.56" y="-154.94"/>
 <instance part="U$22" gate="G$1" x="-381" y="5.08"/>
 <instance part="U$23" gate="G$1" x="-353.06" y="17.78"/>
 <instance part="R11" gate="G$1" x="-393.7" y="-20.32"/>
 <instance part="R12" gate="G$1" x="-360.68" y="-20.32"/>
-<instance part="U$24" gate="G$1" x="-381" y="-91.44"/>
-<instance part="U$25" gate="G$1" x="-381" y="-109.22"/>
+<instance part="U$18" gate="G$1" x="-345.44" y="-93.98"/>
+<instance part="U$19" gate="G$1" x="-345.44" y="-111.76"/>
 </instances>
 <busses>

Commit message: all the traces on top layer alone next will include bottom layer for traces
Parts:
- added U$20: BALL_CASTER, BALL_CASTER:BALL_CASTER
Changed lines of the file:
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@@
 <part name="U$18" library="MOTOR_BRACKET" deviceset="MOTOR_BRACKET" device=""/>
 <part name="U$19" library="MOTOR_BRACKET" deviceset="MOTOR_BRACKET" device=""/>
+<part name="U$20" library="BALL_CASTER" deviceset="BALL_CASTER" device=""/>
 </parts>
 <sheets>
@@
 <instance part="U$18" gate="G$1" x="-345.44" y="-93.98"/>
 <instance part="U$19" gate="G$1" x="-345.44" y="-111.76"/>
+<instance part="U$20" gate="G$1" x="-365.76" y="-73.66"/>
 </instances>
 <busses>
